File: RotaryEncoders.kicad_sch (KiCad schematic)
At the start: 14 parts, among them U5 PEC11H-4025F-S0016, U6 PEC11H-4025F-S0016

Commit message: Major changes
Parts:
- renumbered C7 to C201, C7 to C202, C7 to C203, C7 to C204, R8 to R201, R8 to R202, R8 to R203, R8 to R204, R8 to R205, R8 to R206, R8 to R207, R8 to R208, U5 to U201, U6 to U202

Commit message: Made changes based on Josh's comments & switched to Switched to WS2812B-2020
Parts:
- U201, U202: footprint Adam_Custom_Footprints:PEC11H4025FS0016 -> PEC11H4025FS0016
Changed lines of the file:
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@@
       (effects (font (size 1.27 1.27)))
     )
-    (property "Footprint" "Adam_Custom_Footprints:PEC11H4025FS0016" (at 121.92 130.48 0)
+    (property "Footprint" "PEC11H4025FS0016" (at 121.92 130.48 0)
       (effects (font (size 1.27 1.27)) (justify left top) hide)
     )
@@
       (effects (font (size 1.27 1.27)))
     )
-    (property "Footprint" "Adam_Custom_Footprints:PEC11H4025FS0016" (at 55.88 130.48 0)
-      (effects (font (size 1.27 1.27)) (justify left top) hide)
-    )
+    (property "Footprint" "PEC11H4025FS0016" (at 55.88 130.48 0)
+      (effects (font (size 1.27 1.27)) (justify left top) hide)
+    )
