File: Universal Control Box.kicad_pcb (KiCad board)
At the start: 4 copper layers, 168.2 x 98.8 mm, 88 parts, among them J101 Conn_01x06, J102 Conn_01x07, J103 USB_C_Receptacle_USB2.0, U101 ESP32-WROOM-32, U102 PCF8575DBR (PCF1), U103 XC6220B331MR-G, U201 PEC11H-4025F-S0016, U202 PEC11H-4025F-S0016

Commit message: suggested changes
Parts:
- moved R103 5.46 mm to (173.2, 33.1), turned to 90 degrees
- moved R102 5.40 mm to (160.4, 33.1), turned to -90 degrees
- moved L101 3.89 mm to (173.2, 28.9), turned to -90 degrees
- moved J103 1.74 mm to (166.8, 32.6)
- moved R206 1.58 mm to (219.5, 66.3)
- moved R207 1.56 mm to (229.4, 66.3)
- moved C105 1.11 mm to (170.1, 48.2), turned to 0 degrees
- moved R101 0.87 mm to (101.3, 38.4), turned to 90 degrees
- moved C101 0.82 mm to (102.9, 38.4), turned to -90 degrees
Routing:
- net +3.3V: track 470.7 -> 13.2 mm, vias 12 -> 18
- net +5V: track 617.0 -> 163.8 mm, vias 11 -> 22
- net /IO0: track 36.9 -> 29.2 mm, vias 2 -> 1
- net GND: track 147.8 -> 140.3 mm, vias 51 -> 59
- net /HA_STATUS: track 56.2 -> 50.2 mm
- net /I2C_SDA: track 65.3 -> 69.4 mm
- net /ESP_TX: track 41.1 -> 37.5 mm
- net /EN: track 41.0 -> 37.8 mm, vias 0 -> 1
- net /Rotary Encoders/SW_RSW2: track 137.1 -> 140.2 mm
- net Net-(U202-CHANNEL_1): track 9.81 -> 7.11 mm
- net Net-(U202-CHANNEL_2): track 9.81 -> 7.13 mm
- net /Rotary Encoders/B_RSW2: track 132.2 -> 134.3 mm
- net /OLED_MOSI: track 45.2 -> 43.1 mm
- net Net-(J103-CC1): track 6.23 -> 8.21 mm, vias 2 -> 0
- net Net-(F101-Pad1): track 9.43 -> 7.61 mm
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- added copper zone on B.Cu, net +3.3V
- added copper zone on F.Cu, net +3.3V
- added copper zone on In2.Cu, net +3.3V
- added copper zone on F.Cu, net +5V
- added copper zone on In2.Cu, net +5V
- added copper zone on B.Cu, net GND
- added copper zone on F.Cu, net GND
- added copper zone on F.Cu, net Net-(F101-Pad1)
- removed copper zone on In2.Cu, net GND
