File: KeyCaps.kicad_sch (KiCad schematic)
At the start: 48 parts

Commit message: Included symbols/footprints/3dmodels to repo
Parts:
- SW301, SW302, SW303, SW304, SW305, SW306, SW307, SW308, SW309, SW310, SW311, SW312, SW313, SW314, SW315, SW316: footprint Adam_Custom_Footprints:CherryMX_1.00u_PCB_WS2812B-2020 -> footprints:CherryMX_1.00u_PCB_WS2812B-2020
Changed lines of the file:
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@@
 			)
 		)
-		(property "Footprint" "Adam_Custom_Footprints:CherryMX_1.00u_PCB_WS2812B-2020"
+		(property "Footprint" "footprints:CherryMX_1.00u_PCB_WS2812B-2020"
 			(at 182.88 48.26 0)
 			(effects
@@
 			)
 		)
-		(property "Footprint" "Adam_Custom_Footprints:CherryMX_1.00u_PCB_WS2812B-2020"
+		(property "Footprint" "footprints:CherryMX_1.00u_PCB_WS2812B-2020"
 			(at 146.05 48.26 0)
 			(effects
@@
 			)
 		)
-		(property "Footprint" "Adam_Custom_Footprints:CherryMX_1.00u_PCB_WS2812B-2020"
+		(property "Footprint" "footprints:CherryMX_1.00u_PCB_WS2812B-2020"
 			(at 146.05 17.78 0)
 			(effects
@@
 			)
 		)
-		(property "Footprint" "Adam_Custom_Footprints:CherryMX_1.00u_PCB_WS2812B-2020"
+		(property "Footprint" "footprints:CherryMX_1.00u_PCB_WS2812B-2020"
 			(at 72.39 17.78 0)
 			(effects
@@
 			)
 		)
-		(property "Footprint" "Adam_Custom_Footprints:CherryMX_1.00u_PCB_WS2812B-2020"
+		(property "Footprint" "footprints:CherryMX_1.00u_PCB_WS2812B-2020"
 			(at 35.56 17.78 0)
 			(effects
@@
 			)
 		)
-		(property "Footprint" "Adam_Custom_Footprints:CherryMX_1.00u_PCB_WS2812B-2020"
+		(property "Footprint" "footprints:CherryMX_1.00u_PCB_WS2812B-2020"
 			(at 35.56 48.26 0)
 			(effects
@@
 			)
 		)
-		(property "Footprint" "Adam_Custom_Footprints:CherryMX_1.00u_PCB_WS2812B-2020"
+		(property "Footprint" "footprints:CherryMX_1.00u_PCB_WS2812B-2020"
 			(at 182.88 17.78 0)
 			(effects
@@
 			)
 		)
-		(property "Footprint" "Adam_Custom_Footprints:CherryMX_1.00u_PCB_WS2812B-2020"
+		(property "Footprint" "footprints:CherryMX_1.00u_PCB_WS2812B-2020"
 			(at 219.71 48.26 0)
 			(effects
@@
 			)
 		)
-		(property "Footprint" "Adam_Custom_Footprints:CherryMX_1.00u_PCB_WS2812B-2020"
+		(property "Footprint" "footprints:CherryMX_1.00u_PCB_WS2812B-2020"
 			(at 256.54 48.26 0)
 			(effects
@@
 			)
 		)
-		(property "Footprint" "Adam_Custom_Footprints:CherryMX_1.00u_PCB_WS2812B-2020"
+		(property "Footprint" "footprints:CherryMX_1.00u_PCB_WS2812B-2020"
 			(at 293.37 17.78 0)
 			(effects
@@
 			)
 		)
-		(property "Footprint" "Adam_Custom_Footprints:CherryMX_1.00u_PCB_WS2812B-2020"
+		(property "Footprint" "footprints:CherryMX_1.00u_PCB_WS2812B-2020"
 			(at 109.22 17.78 0)
 			(effects
@@
 			)
 		)
-		(property "Footprint" "Adam_Custom_Footprints:CherryMX_1.00u_PCB_WS2812B-2020"
+		(property "Footprint" "footprints:CherryMX_1.00u_PCB_WS2812B-2020"
 			(at 72.39 48.26 0)
 			(effects
@@
 			)
 		)
-		(property "Footprint" "Adam_Custom_Footprints:CherryMX_1.00u_PCB_WS2812B-2020"
+		(property "Footprint" "footprints:CherryMX_1.00u_PCB_WS2812B-2020"
 			(at 219.71 17.78 0)
 			(effects
@@
 			)
 		)
-		(property "Footprint" "Adam_Custom_Footprints:CherryMX_1.00u_PCB_WS2812B-2020"
+		(property "Footprint" "footprints:CherryMX_1.00u_PCB_WS2812B-2020"
 			(at 293.37 48.26 0)
 			(effects
@@
 			)
 		)
-		(property "Footprint" "Adam_Custom_Footprints:CherryMX_1.00u_PCB_WS2812B-2020"
+		(property "Footprint" "footprints:CherryMX_1.00u_PCB_WS2812B-2020"
 			(at 256.54 17.78 0)
 			(effects
@@
 			)
 		)
-		(property "Footprint" "Adam_Custom_Footprints:CherryMX_1.00u_PCB_WS2812B-2020"
+		(property "Footprint" "footprints:CherryMX_1.00u_PCB_WS2812B-2020"
 			(at 109.22 48.26 0)
 			(effects
