File: Universal Control Box.kicad_sch (KiCad schematic)
At the start: 36 parts, among them J102 Conn_01x07, J103 USB_C_Receptacle_USB2.0, Q101 MMDT3904, U101 ESP32-WROOM-32, U102 PCF8575DBR (PCF1), U103 XC6220B331MR-G, U104 74AHCT1G125, U105 CP2102-GMR

Commit message: Fixed part #s & switched TX & RX
Parts:
- added SW101, SW102: SW_Push, footprints:XKB-Connectivity-TS-1187A-B-A-B, symbol Switch:SW_Push
- C101: LCSC C15849 -> C14663
- C102: LCSC C96446 -> C15850
Connections:
- net EN: now also SW101.1
- net ESP_RX: now also U105.26 (TXD); no longer U105.25 (RXD)
- net ESP_TX: now also U105.25 (RXD); no longer U105.26 (TXD)
- net GND: now also SW101.2, SW102.2
- net IO0: now also SW102.1
Other:
- note added: "Manual Programming (Backup)"

Commit message: Updated PCB to include USB based RX/TX
Parts:
- C106: footprint Capacitor_SMD:C_0805_2012Metric -> Capacitor_SMD:C_0603_1608Metric; LCSC C15850 -> C96446
Changed lines of the file:
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@@
 	(title_block
 		(title "Universal Control Box")
-		(rev "v1.0")
+		(date "2024-06-09")
+		(rev "v2.0")
 	)
 	(junction
@@
 			)
 		)
-		(property "Footprint" "Capacitor_SMD:C_0805_2012Metric"
+		(property "Footprint" "Capacitor_SMD:C_0603_1608Metric"
 			(at 91.44 138.43 0)
 			(effects
@@
 			)
 		)
-		(property "LCSC" "C15850"
+		(property "LCSC" "C96446"
 			(at 91.44 138.43 0)
 			(effects

Commit message: Fixed GND positions & LCSC part for dual mosfet
Parts:
- Q101: LCSC C83572 -> C83572
Changed lines of the file:
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@@
 			)
 		)
-		(property "LCSC" " C83572"
+		(property "LCSC" "C83572"
 			(at 223.52 125.73 0)
 			(effects
@@
 			)
 		)
-		(property "LCSC" " C83572"
+		(property "LCSC" "C83572"
 			(at 223.52 111.76 0)
 			(effects
